Commit message: Robot can controlwoth /cmd_vel command

File: urdf/lidar_bot.xacro (robot description, xacro)
@@ -9,5 +9,5 @@
   <xacro:property name="wheel_length_gap" value="0.05"/>
   <!-- Wheels -->
-  <xacro:macro name="wheel" params="prefix x y wheel_rotate">
+  <xacro:macro name="wheel" params="prefix x y wheel_rotate axix">
     <link name="${prefix}_wheel">
       <visual>
@@ -16,11 +16,4 @@
         </geometry>
         <material name="black"/>
-      </visual>
-      <visual name="${prefix}_wheel_dot">
-        <origin xyz="${wheel_radius} 0 0" rpy="0 0 0"/>
-        <geometry>
-          <sphere radius="0.01"/>
-        </geometry>
-        <material name="red"/>
       </visual>
       <collision>
@@ -31,6 +24,7 @@
       <inertial>
         <origin xyz="0 0 ${wheel_radius}" rpy="0 0 0"/>
-        <mass value="0.5"/>
-        <inertia ixx="0.01" ixy="0" ixz="0" iyy="0.01" iyz="0" izz="0.01"/>
+        <mass value="0.2"/>
+        <!-- <inertia ixx="0.01" ixy="0" ixz="0" iyy="0.01" iyz="0" izz="0.01"/> -->
+        <inertia ixx="0.001633" ixy="0" ixz="0" iyy="0.001633" iyz="0" izz="0.0016"/>
       </inertial>
     </link>
@@ -39,6 +33,6 @@
       <child link="${prefix}_wheel"/>
       <origin xyz="${x} ${y} 0" rpy="${wheel_rotate} 0 0"/>
-      <limit effort="10" velocity="5" lower="-3.14" upper="3.14"/>
-      <axis xyz="0 0 1"/>
+      <limit effort="50" velocity="20" lower="-3.14" upper="3.14"/>
+      <axis xyz="0 0 ${axix}"/>
       <dynamics damping="0.1" friction="0.1"/>
       <safety_controller soft_lower_limit="-1.0" soft_upper_limit="1.0" k_position="100" k_velocity="10"/>
@@ -80,6 +74,4 @@
     <color rgba="1.0 0.2 0.6 1"/>
   </material>
-  <!-- World link -->
-  <link name="world"/>
   <!-- Base Link -->
   <link name="base_link">
@@ -91,4 +83,5 @@
     </visual>
     <collision>
+      <origin xyz="0 0 ${wheel_radius/2}"/>
       <geometry>
         <box size="${body_length} ${body_width} ${body_height}"/>
@@ -96,62 +89,46 @@
     </collision>
     <inertial>
-      <mass value="5"/>
-      <inertia ixx="0.1" ixy="0" ixz="0" iyy="0.1" iyz="0" izz="0.1"/>
+      <mass value="0.5"/>
+      <inertia ixx="0.04167" ixy="0" ixz="0" iyy="0.07083" iyz="0" izz="0.10417"/>
     </inertial>
   </link>
-  <!-- World to base joint -->
-  <joint name="base_to_world" type="fixed">
-    <parent link="world"/>
-    <child link="base_link"/>
-    <origin xyz="0 0 ${body_height + wheel_radius}" rpy="0 0 0"/>
-  </joint>
   <!-- Wheels -->
-  <xacro:wheel prefix="left_front" x="${body_length/2 - wheel_length_gap}" y="${body_width/2 + wheel_width/2}" wheel_rotate="1.57"/>
-  <xacro:wheel prefix="left_rear" x="-${body_length/2 - wheel_length_gap}" y="${body_width/2 + wheel_width/2}" wheel_rotate="1.57"/>
-  <xacro:wheel prefix="right_front" x="${body_length/2 - wheel_length_gap}" y="-${body_width/2 + wheel_width/2}" wheel_rotate="1.57"/>
-  <xacro:wheel prefix="right_rear" x="-${body_length/2 - wheel_length_gap}" y="-${body_width/2 + wheel_width/2}" wheel_rotate="1.57"/>
+  <xacro:wheel prefix="left_front" x="-${body_length/2 - wheel_length_gap}" y="${body_width/2 + wheel_width/2}" wheel_rotate="-1.570796" axix="1"/>
+  <xacro:wheel prefix="left_rear" x="${body_length/2 - wheel_length_gap}" y="${body_width/2 + wheel_width/2}" wheel_rotate="-1.570796" axix="1"/>
+  <xacro:wheel prefix="right_front" x="-${body_length/2 - wheel_length_gap}" y="-${body_width/2 + wheel_width/2}" wheel_rotate="1.570796" axix="-1"/>
+  <xacro:wheel prefix="right_rear" x="${body_length/2 - wheel_length_gap}" y="-${body_width/2 + wheel_width/2}" wheel_rotate="1.570796" axix="-1"/>
   <gazebo reference="base_link">
-    <mu1>0.8</mu1>
-    <mu2>0.8</mu2>
+    <mu1>1.0</mu1>
+    <mu2>1.0</mu2>
     <material>Gazebo/Blue</material>
   </gazebo>
   <gazebo reference="left_front_wheel">
-    <mu1>0.8</mu1>
-    <mu2>0.8</mu2>
+    <mu1>1.0</mu1>
+    <mu2>1.0</mu2>
+    <kp>1000000.0</kp>
+    <kd>1.0</kd>
     <material>Gazebo/Black</material>
   </gazebo>
   <gazebo reference="left_rear_wheel">
-    <mu1>0.8</mu1>
-    <mu2>0.8</mu2>
+    <mu1>1.0</mu1>
+    <mu2>1.0</mu2>
+    <kp>1000000.0</kp>
+    <kd>1.0</kd>
+    <material>Gazebo/Green</material>
+  </gazebo>
+  <gazebo reference="right_front_wheel">
+    <mu1>1.0</mu1>
+    <mu2>1.0</mu2>
+    <kp>1000000.0</kp>
+    <kd>1.0</kd>
     <material>Gazebo/Black</material>
   </gazebo>
-  <gazebo reference="right_front_wheel">
-    <mu1>0.8</mu1>
-    <mu2>0.8</mu2>
-    <material>Gazebo/Black</material>
-  </gazebo>
   <gazebo reference="right_rear_wheel">
-    <mu1>0.8</mu1>
-    <mu2>0.8</mu2>
-    <material>Gazebo/Black</material>
-  </gazebo>
-<!-- Plugin to simulate differential drive -->
-<!-- <gazebo>
-  <plugin name="diff_drive_controller" filename="libgazebo_ros_diff_drive.so">
-    <ros>
-      <namespace>/</namespace>
-      <remapping>cmd_vel:=/cmd_vel</remapping>
-    </ros>
-    <left_joint>left_front_wheel_joint</left_joint>
-    <left_joint>left_rear_wheel_joint</left_joint>
-    <right_joint>right_front_wheel_joint</right_joint>
-    <right_joint>right_rear_wheel_joint</right_joint>
-    <wheel_separation>0.34</wheel_separation>
-    <wheel_diameter>0.16</wheel_diameter>
-    <broadcast_tf>true</broadcast_tf>
-    <publish_odom>true</publish_odom>
-    <robot_base_frame>base_link</robot_base_frame>
-  </plugin>
-</gazebo> -->
+    <mu1>1.0</mu1>
+    <mu2>1.0</mu2>
+    <kp>1000000.0</kp>
+    <kd>1.0</kd>
+    <material>Gazebo/Green</material>
+  </gazebo>
   <!-- left_front_wheel -->
   <transmission name="left_front_wheel_trans">
@@ -164,4 +141,7 @@
     </actuator>
   </transmission>
+  <gazebo reference="left_front_wheel_joint">
+    <provideFeedback>true</provideFeedback>
+  </gazebo>
   <!-- left_rear_wheel -->
   <transmission name="left_rear_wheel_trans">
@@ -174,4 +154,7 @@
     </actuator>
   </transmission>
+  <gazebo reference="left_rear_wheel_joint">
+    <provideFeedback>true</provideFeedback>
+  </gazebo>
   <!-- right_front_wheel -->
   <transmission name="right_front_wheel_trans">
@@ -184,4 +167,7 @@
     </actuator>
   </transmission>
+  <gazebo reference="right_front_wheel_joint">
+    <provideFeedback>true</provideFeedback>
+  </gazebo>
   <!-- right_rear_wheel -->
   <transmission name="right_rear_wheel_trans">
@@ -194,14 +180,9 @@
     </actuator>
   </transmission>
-  <!-- <gazebo reference="right_rear_wheel">
-    <mu1>0.8</mu1>
-    <mu2>0.8</mu2>
-    <material>Gazebo/Black</material>
-  </gazebo>
   <gazebo reference="right_rear_wheel_joint">
     <provideFeedback>true</provideFeedback>
-  </gazebo> -->
+  </gazebo>
   <!-- LiDAR Sensor (Hokuyo style) -->
-  <!-- <link name="laser">
+  <link name="laser_link">
     <visual>
       <geometry>
@@ -214,7 +195,10 @@
   <joint name="laser_joint" type="fixed">
     <parent link="base_link"/>
-    <child link="laser"/>
+    <child link="laser_link"/>
     <origin xyz="0 0 ${body_height/2}" rpy="0 0 0"/>
-  </joint> -->
+  </joint>
+  <gazebo reference="laser_link">
+    <material>Gazebo/neon_pink</material>
+  </gazebo>
   <!-- Plugin to load ros_control -->
   <gazebo>
@@ -223,10 +207,6 @@
     </plugin>
     <plugin name="diff_drive_controller" filename="libgazebo_ros_diff_drive.so">
-      <updateRate>100.0</updateRate>
+      <updateRate>50.0</updateRate>
       <robotNamespace>/</robotNamespace>
-      <!-- <left_wheel>left_front_wheel</left_wheel> -->
-      <!-- <left_wheel>left_rear_wheel</left_wheel> -->
-      <!-- <right_wheel>right_front_wheel</right_wheel> -->
-      <!-- <right_wheel>right_rear_wheel</right_wheel> -->
       <leftJoint>left_front_wheel_joint</leftJoint>
       <leftJoint>left_rear_wheel_joint</leftJoint>
@@ -240,9 +220,8 @@
       <publishOdomTF>true</publishOdomTF>
       <publishWheelJointState>true</publishWheelJointState>
-      <wheelAcceleration>0.5</wheelAcceleration>
-      <wheelTorque>5</wheelTorque>
-      <odometrySource>1</odometrySource>
+      <wheelAcceleration>1.0</wheelAcceleration>
+      <wheelTorque>20</wheelTorque>
+      <odometrySource>odom</odometrySource>
       <publishTf>1</publishTf>
-      <torque>50</torque>
       <commandTopic>cmd_vel</commandTopic>
       <odometryTopic>odom</odometryTopic>

Commit message: Updated

File: urdf/lidar_bot.xacro (robot description, xacro)
@@ -33,5 +33,5 @@
       <child link="${prefix}_wheel"/>
       <origin xyz="${x} ${y} 0" rpy="${wheel_rotate} 0 0"/>
-      <limit effort="50" velocity="20" lower="-3.14" upper="3.14"/>
+      <limit effort="50" velocity="20" lower="-100" upper="100"/>
       <axis xyz="0 0 ${axix}"/>
       <dynamics damping="0.1" friction="0.1"/>
@@ -94,8 +94,8 @@
   </link>
   <!-- Wheels -->
-  <xacro:wheel prefix="left_front" x="-${body_length/2 - wheel_length_gap}" y="${body_width/2 + wheel_width/2}" wheel_rotate="-1.570796" axix="1"/>
-  <xacro:wheel prefix="left_rear" x="${body_length/2 - wheel_length_gap}" y="${body_width/2 + wheel_width/2}" wheel_rotate="-1.570796" axix="1"/>
-  <xacro:wheel prefix="right_front" x="-${body_length/2 - wheel_length_gap}" y="-${body_width/2 + wheel_width/2}" wheel_rotate="1.570796" axix="-1"/>
-  <xacro:wheel prefix="right_rear" x="${body_length/2 - wheel_length_gap}" y="-${body_width/2 + wheel_width/2}" wheel_rotate="1.570796" axix="-1"/>
+  <xacro:wheel prefix="left_front" x="-${body_length/2 - wheel_length_gap}" y="${body_width/2 + wheel_width/2}" wheel_rotate="-1.570796" axix="-1"/>
+  <xacro:wheel prefix="left_rear" x="${body_length/2 - wheel_length_gap}" y="${body_width/2 + wheel_width/2}" wheel_rotate="-1.570796" axix="-1"/>
+  <xacro:wheel prefix="right_front" x="-${body_length/2 - wheel_length_gap}" y="-${body_width/2 + wheel_width/2}" wheel_rotate="1.570796" axix="1"/>
+  <xacro:wheel prefix="right_rear" x="${body_length/2 - wheel_length_gap}" y="-${body_width/2 + wheel_width/2}" wheel_rotate="1.570796" axix="1"/>
   <gazebo reference="base_link">
     <mu1>1.0</mu1>
@@ -106,4 +106,8 @@
     <mu1>1.0</mu1>
     <mu2>1.0</mu2>
+    <dynamics>
+      <friction>5.0</friction>
+      <damping>0.7</damping>
+    </dynamics>
     <kp>1000000.0</kp>
     <kd>1.0</kd>
@@ -113,4 +117,8 @@
     <mu1>1.0</mu1>
     <mu2>1.0</mu2>
+    <dynamics>
+      <friction>5.0</friction>
+      <damping>0.7</damping>
+    </dynamics>
     <kp>1000000.0</kp>
     <kd>1.0</kd>
@@ -120,4 +128,8 @@
     <mu1>1.0</mu1>
     <mu2>1.0</mu2>
+    <dynamics>
+      <friction>5.0</friction>
+      <damping>0.7</damping>
+    </dynamics>
     <kp>1000000.0</kp>
     <kd>1.0</kd>
@@ -127,4 +139,8 @@
     <mu1>1.0</mu1>
     <mu2>1.0</mu2>
+    <dynamics>
+      <friction>5.0</friction>
+      <damping>0.7</damping>
+    </dynamics>
     <kp>1000000.0</kp>
     <kd>1.0</kd>
@@ -207,5 +223,5 @@
     </plugin>
     <plugin name="diff_drive_controller" filename="libgazebo_ros_diff_drive.so">
-      <updateRate>50.0</updateRate>
+      <updateRate>100.0</updateRate>
       <robotNamespace>/</robotNamespace>
       <leftJoint>left_front_wheel_joint</leftJoint>
@@ -221,5 +237,5 @@
       <publishWheelJointState>true</publishWheelJointState>
       <wheelAcceleration>1.0</wheelAcceleration>
-      <wheelTorque>20</wheelTorque>
+      <wheelTorque>15</wheelTorque>
       <odometrySource>odom</odometrySource>
       <publishTf>1</publishTf>

Commit message: updated

File: urdf/lidar_bot.xacro (robot description, xacro)
@@ -115,8 +115,8 @@
   </gazebo>
   <gazebo reference="left_rear_wheel">
-    <mu1>1.0</mu1>
-    <mu2>1.0</mu2>
-    <dynamics>
-      <friction>5.0</friction>
+    <mu1>0.1</mu1>
+    <mu2>0.1</mu2>
+    <dynamics>
+      <friction>1.0</friction>
       <damping>0.7</damping>
     </dynamics>
@@ -137,13 +137,13 @@
   </gazebo>
   <gazebo reference="right_rear_wheel">
-    <mu1>1.0</mu1>
-    <mu2>1.0</mu2>
-    <dynamics>
-      <friction>5.0</friction>
-      <damping>0.7</damping>
-    </dynamics>
-    <kp>1000000.0</kp>
-    <kd>1.0</kd>
-    <material>Gazebo/Green</material>
+    <mu1>0.1</mu1>
+    <mu2>0.1</mu2>
+    <dynamics>
+      <friction>1.0</friction>
+      <damping>0.7</damping>
+    </dynamics>
+    <kp>1000000.0</kp>
+    <kd>1.0</kd>
+    <material>Gazebo/Red</material>
   </gazebo>
   <!-- left_front_wheel -->
@@ -200,5 +200,5 @@
   </gazebo>
   <!-- LiDAR Sensor (Hokuyo style) -->
-  <link name="laser_link">
+  <!-- <link name="laser_link">
     <visual>
       <geometry>
@@ -216,5 +216,5 @@
   <gazebo reference="laser_link">
     <material>Gazebo/neon_pink</material>
-  </gazebo>
+  </gazebo> -->
   <!-- Plugin to load ros_control -->
   <gazebo>
@@ -226,7 +226,7 @@
       <robotNamespace>/</robotNamespace>
       <leftJoint>left_front_wheel_joint</leftJoint>
-      <leftJoint>left_rear_wheel_joint</leftJoint>
+      <!-- <leftJoint>left_rear_wheel_joint</leftJoint> -->
       <rightJoint>right_front_wheel_joint</rightJoint>
-      <rightJoint>right_rear_wheel_joint</rightJoint>
+      <!-- <rightJoint>right_rear_wheel_joint</rightJoint> -->
       <wheelSeparation>0.32</wheelSeparation>
       <wheelDiameter>0.16</wheelDiameter>
