Commit message: Update odom slam navigation codes

File: urdf/gazebo.xacro (robot description, xacro)
@@ -23,4 +23,5 @@
       <updateRate>50</updateRate>
       <max_velocity>0.5</max_velocity>
+      <rosDebugLevel>0</rosDebugLevel>
     </plugin>
   </gazebo>

File: urdf/lidar_scanning_robot.xacro (robot description, xacro)
@@ -9,5 +9,5 @@
   <xacro:include filename="$(find lidar_scanning_robot)/urdf/gazebo.xacro" />
   <!-- Include Lidar -->
-  <!-- <xacro:include filename="$(find lidar_scanning_robot)/urdf/lidar.xacro" /> -->
+  <xacro:include filename="$(find lidar_scanning_robot)/urdf/lidar.xacro" />
   <!-- Base Link -->
   <link name="base_link">

File: urdf/macros.xacro (robot description, xacro)
@@ -25,5 +25,5 @@
       <parent link="base_link"/>
       <child link="${prefix}_wheel"/>
-      <origin xyz="${x} ${y * (base_width/2 + wheel_radius/2)} 0" rpy="${pi/2} 0 0"/>  <!-- Corrected RPY and Z offset -->
+      <origin xyz="${x} ${y * (base_width/2 + wheel_radius/2)} 0" rpy="${pi/2} 0 0"/>
       <axis xyz="0 0 -1"/>
       <joint_properties damping="0.5" friction="0.5"/>
